File: hardware/controller/RP2040_Zero_Carrier.kicad_pcb (KiCad board)
At the start: 2 copper layers, 40 x 36 mm, 6 parts, among them J1 20P 1.0mm FFC ZIF bottom-cont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, U1 Waveshare RP2040-Zero

Commit message: Finalize FFC routing and assembly-safe hardware
Routing:
- net COL12: track 32.9 -> 30.1 mm
- net ROW4: track 28.6 -> 25.8 mm
- net ROW2: track 32.5 -> 29.7 mm
- net ROW1: track 34.0 -> 31.2 mm
- net ROW0: track 34.8 -> 32.0 mm
- net GND: track 42.6 -> 39.8 mm
- net COL9: track 28.3 -> 25.5 mm
- net COL8: track 28.4 -> 25.6 mm
- net COL4: track 16.1 -> 13.3 mm
- net COL3: track 14.9 -> 12.1 mm
- net COL2: track 14.2 -> 11.4 mm
- net COL13: track 34.6 -> 31.8 mm
- net COL11: track 32.1 -> 29.3 mm
- net COL10: track 30.6 -> 27.8 mm
- net COL1: track 13.2 -> 10.4 mm
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Changed lines of the file:
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@@
 		(at 0 0)
 		(property "Reference" "J1"
-			(at 20 37.6 0)
+			(at 20 34.8 0)
 			(layer "B.Fab")
 			(effects
@@
 		)
 		(property "Value" "20P 1.0mm FFC ZIF bottom-contact"
-			(at 20 32.8 0)
+			(at 20 30 0)
 			(layer "B.Fab")
 			(hide yes)
@@
 		(duplicate_pad_numbers_are_jumpers no)
 		(fp_line
-			(start 9 29.6)
-			(end 31 29.6)
+			(start 9 26.8)
+			(end 31 26.8)
 			(stroke
 				(width 0.5)
@@
 		)
 		(fp_rect
-			(start 8.4 28.8)
-			(end 31.6 35.8)
+			(start 8.4 26)
+			(end 31.6 33)
 			(stroke
 				(width 0.25)
@@
 		)
 		(pad "" smd rect
-			(at 8.7 33.5)
+			(at 8.7 30.7)
 			(size 2.4 3.2)
 			(layers "B.Cu" "B.Mask" "B.Paste")
 		)
 		(pad "" smd rect
-			(at 31.3 33.5)
+			(at 31.3 30.7)
 			(size 2.4 3.2)
 			(layers "B.Cu" "B.Mask" "B.Paste")
 		)
 		(pad "1" smd roundrect
-			(at 10.5 32.8)
+			(at 10.5 30)
 			(size 0.6 2.6)
 			(layers "B.Cu" "B.Mask" "B.Paste")
@@
 		)
 		(pad "2" smd roundrect
-			(at 11.5 32.8)
+			(at 11.5 30)
 			(size 0.6 2.6)
 			(layers "B.Cu" "B.Mask" "B.Paste")
@@
 		)
 		(pad "3" smd roundrect
-			(at 12.5 32.8)
+			(at 12.5 30)
 			(size 0.6 2.6)
 			(layers "B.Cu" "B.Mask" "B.Paste")
@@
 		)
 		(pad "4" smd roundrect
-			(at 13.5 32.8)
+			(at 13.5 30)
 			(size 0.6 2.6)
 			(layers "B.Cu" "B.Mask" "B.Paste")
@@
 		)
 		(pad "5" smd roundrect
-			(at 14.5 32.8)
+			(at 14.5 30)
 			(size 0.6 2.6)
 			(layers "B.Cu" "B.Mask" "B.Paste")
@@
 		)
 		(pad "6" smd roundrect
-			(at 15.5 32.8)
+			(at 15.5 30)
 			(size 0.6 2.6)
 			(layers "B.Cu" "B.Mask" "B.Paste")
@@
 		)
 		(pad "7" smd roundrect
-			(at 16.5 32.8)
+			(at 16.5 30)
 			(size 0.6 2.6)
 			(layers "B.Cu" "B.Mask" "B.Paste")
@@
 		)
 		(pad "8" smd roundrect
-			(at 17.5 32.8)
+			(at 17.5 30)
 			(size 0.6 2.6)
 			(layers "B.Cu" "B.Mask" "B.Paste")
@@
 		)
 		(pad "9" smd roundrect
-			(at 18.5 32.8)
+			(at 18.5 30)
 			(size 0.6 2.6)
 			(layers "B.Cu" "B.Mask" "B.Paste")
@@
 		)
 		(pad "10" smd roundrect
-			(at 19.5 32.8)
+			(at 19.5 30)
 			(size 0.6 2.6)
 			(layers "B.Cu" "B.Mask" "B.Paste")
@@
 		)
 		(pad "11" smd roundrect
-			(at 20.5 32.8)
+			(at 20.5 30)
 			(size 0.6 2.6)
 			(layers "B.Cu" "B.Mask" "B.Paste")
@@
 		)
 		(pad "12" smd roundrect
-			(at 21.5 32.8)
+			(at 21.5 30)
 			(size 0.6 2.6)
 			(layers "B.Cu" "B.Mask" "B.Paste")
@@
 		)
 		(pad "13" smd roundrect
-			(at 22.5 32.8)
+			(at 22.5 30)
 			(size 0.6 2.6)
 			(layers "B.Cu" "B.Mask" "B.Paste")
@@
 		)
 		(pad "14" smd roundrect
-			(at 23.5 32.8)
+			(at 23.5 30)
 			(size 0.6 2.6)
 			(layers "B.Cu" "B.Mask" "B.Paste")
@@
 		)
 		(pad "15" smd roundrect
-			(at 24.5 32.8)
+			(at 24.5 30)
 			(size 0.6 2.6)
 			(layers "B.Cu" "B.Mask" "B.Paste")
@@
 		)
 		(pad "16" smd roundrect
-			(at 25.5 32.8)
+			(at 25.5 30)
 			(size 0.6 2.6)
 			(layers "B.Cu" "B.Mask" "B.Paste")
@@
 		)
 		(pad "17" smd roundrect
-			(at 26.5 32.8)
+			(at 26.5 30)
 			(size 0.6 2.6)
 			(layers "B.Cu" "B.Mask" "B.Paste")
@@
 		)
 		(pad "18" smd roundrect
-			(at 27.5 32.8)
+			(at 27.5 30)
 			(size 0.6 2.6)
 			(layers "B.Cu" "B.Mask" "B.Paste")
@@
 		)
 		(pad "19" smd roundrect
-			(at 28.5 32.8)
+			(at 28.5 30)
 			(size 0.6 2.6)
 			(layers "B.Cu" "B.Mask" "B.Paste")
@@
 		)
 		(pad "20" smd roundrect
-			(at 29.5 32.8)
+			(at 29.5 30)
 			(size 0.6 2.6)
 			(layers "B.Cu" "B.Mask" "B.Paste")
@@
 	)
 	(segment
-		(start 10.5 32.8)
+		(start 10.5 30)
 		(end 10.5 25.5235)
 		(width 0.2)
@@
 	)
 	(segment
-		(start 11.5 32.8)
+		(start 11.5 30)
 		(end 11.5 26.3164)
 		(width 0.2)
@@
 	)
 	(segment
-		(start 12.5 32.8)
+		(start 12.5 30)
 		(end 12.5 26.9265)
 		(width 0.2)
@@
 	)
 	(segment
-		(start 13.5 32.8)
+		(start 13.5 30)
 		(end 13.5 28.292)
 		(width 0.2)
@@
 	)
 	(segment
-		(start 14.5 32.8)
+		(start 14.5 30)
 		(end 14.5 28.9096)
 		(width 0.2)
@@
 	(segment
 		(start 22.8987 29.5113)
-		(end 17.0374 29.5113)
+		(end 15.5 29.5113)
 		(width 0.2)
 		(layer "F.Cu")
@@
 	)
 	(via
-		(at 17.0374 29.5113)
+		(at 15.5 29.5113)
 		(size 0.6)
 		(drill 0.3)
@@
 	)
 	(segment
-		(start 16.2018 29.5113)
-		(end 17.0374 29.5113)
-		(width 0.2)
-		(layer "B.Cu")
-		(net "COL5")
-	)
-	(segment
-		(start 15.5 32.8)
-		(end 15.5 30.2131)
-		(width 0.2)
-		(layer "B.Cu")
-		(net "COL5")
-	)
-	(segment
-		(start 15.5 30.2131)
-		(end 16.2018 29.5113)
+		(start 15.5 30)
+		(end 15.5 29.5113)
 		(width 0.2)
 		(layer "B.Cu")
@@
 	)
 	(segment
-		(start 16.5 32.8)
+		(start 16.5 30)
 		(end 16.5 30.113)
 		(width 0.2)
@@
 	)
 	(segment
-		(start 17.5 32.8)
+		(start 17.5 30)
 		(end 17.7588 32.5412)
 		(width 0.2)
@@
 	)
 	(segment
-		(start 18.5 32.8)
+		(start 18.5 30)
 		(end 18.5 15.1731)
 		(width 0.2)
@@
 	)
 	(segment
-		(start 19.5 32.8)
+		(start 19.5 30)
 		(end 19.5 14.4477)
 		(width 0.2)
@@
 	)
 	(segment
-		(start 20.5 32.8)
+		(start 20.5 30)
 		(end 20.5 10.71)
 		(width 0.2)
@@
 	)
 	(segment
-		(start 21.5 32.8)
+		(start 21.5 30)
 		(end 21.5 8.17)
 		(width 0.2)
@@
 	)
 	(segment
-		(start 22.5 32.8)
+		(start 22.5 30)
 		(end 22.5 6.8606)
 		(width 0.2)
@@
 	)
 	(segment
-		(start 23.5 32.8)
+		(start 23.5 30)
 		(end 23.5 4.0759)
 		(width 0.2)
@@
 	)
 	(segment
-		(start 24.5 32.8)
+		(start 24.5 30)
 		(end 24.5 12.1174)
 		(width 0.2)
@@
 	)
 	(segment
-		(start 25.5 32.8)
+		(start 25.5 30)
 		(end 25.5 13.25)
 		(width 0.2)
@@
 	)
 	(segment
-		(start 26.5 32.8)
+		(start 26.5 30)
 		(end 26.5 15.8748)
 		(width 0.2)
@@
 	)
 	(segment
-		(start 27.5 32.8)
+		(start 27.5 30)
 		(end 27.5 22.14)
 		(width 0.2)
@@
 	)
 	(segment
-		(start 28.5 32.8)
+		(start 28.5 30)
 		(end 28.5 22.2571)
 		(width 0.2)
@@
 	)
 	(segment
-		(start 29.5 32.8)
+		(start 29.5 30)
 		(end 29.5 10.9426)
 		(width 0.2)
